File: kicad/TT1a/TT1a.kicad_sch (KiCad schematic)
At the start: 14 parts, among them SW1 SW_Push, SW2 SW_Push, SW3 SW_Push, SW4 SW_Push, U1 ATtiny404-SS

Commit message: Schematic done but components arent done yet Bat1: use BAT-HLD-001 Switches: use PTS526 SK15 SMTR2 LFS update library for that
Parts:
- added C1: 10uF, Capacitor_SMD:C_0805_2012Metric, symbol Device:C
- added C2: 100nF, Capacitor_SMD:C_0603_1608Metric, symbol Device:C
- added TP1, TP2, TP3, TP4, TP5, TP6: TestPoint, TestPoint:TestPoint_Pad_D1.0mm, symbol Connector:TestPoint
- BT1: footprint (none) -> Battery:BatteryHolder_LINX_BAT-HLD-012-SMT
- D1, D2, D3, D4: footprint (none) -> LED_SMD:LED_0603_1608Metric
- R1, R2, R3, R4: value R -> 1k; footprint (none) -> Resistor_SMD:R_0603_1608Metric
- SW1, SW2, SW3, SW4: footprint (none) -> Button_Switch_SMD:SW_SPST_PTS645
Connections:
- net +BATT: now also U1.1 (VCC), C1.1, C2.1, TP1.1
- net BTN1: now also U1.9 (PB0)
- net BTN2: now also U1.8 (PB1)
- net BTN3: now also U1.7 (PB2)
- net BTN4: now also U1.6 (PB3)
- net GND: now also C1.2, C2.2, TP2.1
- net LED1: now also U1.2 (PA4)
- net LED2: now also U1.3 (PA5)
- net LED3: now also U1.4 (PA6)
- net LED4: now also U1.5 (PA7)
- net at U1.10 (~{RESET}/PA0): now also TP3.1
- net at U1.11 (PA1): now also TP4.1
- net at U1.12 (PA2): now also TP5.1
- net at U1.13 (PA3): now also TP6.1

Commit message: TT1a: changed footprints for Bat + Buttons
Parts:
- BT1: footprint Battery:BatteryHolder_LINX_BAT-HLD-012-SMT -> MEgli:BAT-HLD-001
- SW1, SW2, SW3, SW4: footprint Button_Switch_SMD:SW_SPST_PTS645 -> MEgli:PTS526_button
Changed lines of the file:
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@@
       (effects (font (size 1.27 1.27)) (justify left))
     )
-    (property "Footprint" "Battery:BatteryHolder_LINX_BAT-HLD-012-SMT" (at 33.02 81.026 90)
+    (property "Footprint" "MEgli:BAT-HLD-001" (at 33.02 81.026 90)
       (effects (font (size 1.27 1.27)) hide)
     )
@@
       (effects (font (size 1.27 1.27)) (justify left))
     )
-    (property "Footprint" "Button_Switch_SMD:SW_SPST_PTS645" (at 266.7 59.69 0)
+    (property "Footprint" "MEgli:PTS526_button" (at 266.7 59.69 0)
       (effects (font (size 1.27 1.27)) hide)
     )
@@
       (effects (font (size 1.27 1.27)) (justify left))
     )
-    (property "Footprint" "Button_Switch_SMD:SW_SPST_PTS645" (at 209.55 59.69 0)
+    (property "Footprint" "MEgli:PTS526_button" (at 209.55 59.69 0)
       (effects (font (size 1.27 1.27)) hide)
     )
@@
       (effects (font (size 1.27 1.27)) (justify left))
     )
-    (property "Footprint" "Button_Switch_SMD:SW_SPST_PTS645" (at 238.76 59.69 0)
+    (property "Footprint" "MEgli:PTS526_button" (at 238.76 59.69 0)
       (effects (font (size 1.27 1.27)) hide)
     )
@@
       (effects (font (size 1.27 1.27)) (justify left))
     )
-    (property "Footprint" "Button_Switch_SMD:SW_SPST_PTS645" (at 180.34 59.69 0)
-      (effects (font (size 1.27 1.27)) hide)
-    )
+    (property "Footprint" "MEgli:PTS526_button" (at 180.34 59.69 0)
+      (effects (font (size 1.27 1.27)) hide)
+    )

Commit message: pcb TT1a done
Connections:
- net BTN1: now also U1.3 (PA5); no longer U1.9 (PB0)
- net BTN2: now also U1.2 (PA4); no longer U1.8 (PB1)
- net LED1: now also U1.13 (PA3); no longer U1.2 (PA4)
- net LED2: now also U1.12 (PA2); no longer U1.3 (PA5)
- net LED3: now also U1.9 (PB0); no longer U1.4 (PA6)
- net LED4: now also U1.8 (PB1); no longer U1.5 (PA7)
- net at TP5.1: now also U1.4 (PA6); no longer U1.12 (PA2)
- net at TP6.1: now also U1.5 (PA7); no longer U1.13 (PA3)
Other:
- moved on the sheet: TP5, TP6
Changed lines of the file:
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@@
     (effects (font (size 1.27 1.27)) (justify right bottom))
   )
-  (label "LED2" (at 109.22 81.28 0) (fields_autoplaced)
+  (label "LED2" (at 109.22 73.66 0) (fields_autoplaced)
     (effects (font (size 1.27 1.27)) (justify left bottom))
   )
@@
     (effects (font (size 1.27 1.27)) (justify left bottom))
   )
-  (label "BTN2" (at 72.39 71.12 180) (fields_autoplaced)
+  (label "BTN2" (at 109.22 78.74 0) (fields_autoplaced)
+    (effects (font (size 1.27 1.27)) (justify left bottom))
+  )
+  (label "LED1" (at 163.83 49.53 0) (fields_autoplaced)
+    (effects (font (size 1.27 1.27)) (justify left bottom))
+  )
+  (label "LED1" (at 109.22 76.2 0) (fields_autoplaced)
+    (effects (font (size 1.27 1.27)) (justify left bottom))
+  )
+  (label "LED3" (at 222.25 49.53 0) (fields_autoplaced)
+    (effects (font (size 1.27 1.27)) (justify left bottom))
+  )
+  (label "BTN1" (at 175.26 49.53 0) (fields_autoplaced)
+    (effects (font (size 1.27 1.27)) (justify left bottom))
+  )
+  (label "LED4" (at 72.39 71.12 180) (fields_autoplaced)
     (effects (font (size 1.27 1.27)) (justify right bottom))
   )
-  (label "LED1" (at 163.83 49.53 0) (fields_autoplaced)
-    (effects (font (size 1.27 1.27)) (justify left bottom))
-  )
-  (label "LED1" (at 109.22 78.74 0) (fields_autoplaced)
-    (effects (font (size 1.27 1.27)) (justify left bottom))
-  )
-  (label "LED3" (at 222.25 49.53 0) (fields_autoplaced)
-    (effects (font (size 1.27 1.27)) (justify left bottom))
-  )
-  (label "BTN1" (at 175.26 49.53 0) (fields_autoplaced)
-    (effects (font (size 1.27 1.27)) (justify left bottom))
-  )
-  (label "LED4" (at 109.22 86.36 0) (fields_autoplaced)
-    (effects (font (size 1.27 1.27)) (justify left bottom))
-  )
   (label "BTN2" (at 204.47 49.53 0) (fields_autoplaced)
     (effects (font (size 1.27 1.27)) (justify left bottom))
   )
-  (label "BTN1" (at 72.39 68.58 180) (fields_autoplaced)
+  (label "BTN1" (at 109.22 81.28 0) (fields_autoplaced)
+    (effects (font (size 1.27 1.27)) (justify left bottom))
+  )
+  (label "LED4" (at 250.19 49.53 0) (fields_autoplaced)
+    (effects (font (size 1.27 1.27)) (justify left bottom))
+  )
+  (label "BTN4" (at 261.62 49.53 0) (fields_autoplaced)
+    (effects (font (size 1.27 1.27)) (justify left bottom))
+  )
+  (label "LED2" (at 193.04 49.53 0) (fields_autoplaced)
+    (effects (font (size 1.27 1.27)) (justify left bottom))
+  )
+  (label "LED3" (at 72.39 68.58 180) (fields_autoplaced)
     (effects (font (size 1.27 1.27)) (justify right bottom))
-  )
-  (label "LED4" (at 250.19 49.53 0) (fields_autoplaced)
-    (effects (font (size 1.27 1.27)) (justify left bottom))
-  )
-  (label "BTN4" (at 261.62 49.53 0) (fields_autoplaced)
-    (effects (font (size 1.27 1.27)) (justify left bottom))
-  )
-  (label "LED2" (at 193.04 49.53 0) (fields_autoplaced)
-    (effects (font (size 1.27 1.27)) (justify left bottom))
-  )
-  (label "LED3" (at 109.22 83.82 0) (fields_autoplaced)
-    (effects (font (size 1.27 1.27)) (justify left bottom))
   )
   (symbol (lib_id "MCU_Microchip_ATtiny:ATtiny404-SS") (at 90.17 78.74 0) (unit 1)
@@
     )
   )
-  (symbol (lib_id "Connector:TestPoint") (at 109.22 76.2 270) (unit 1)
+  (symbol (lib_id "Connector:TestPoint") (at 109.22 86.36 270) (unit 1)
     (in_bom yes) (on_board yes) (dnp no)
-    (property "Reference" "TP6" (at 114.3 75.565 90)
-      (effects (font (size 1.27 1.27)) (justify left))
-    )
-    (property "Value" "TestPoint" (at 118.11 76.2 90)
+    (property "Reference" "TP6" (at 114.3 85.725 90)
+      (effects (font (size 1.27 1.27)) (justify left))
+    )
+    (property "Value" "TestPoint" (at 118.11 86.36 90)
       (effects (font (size 1.27 1.27)) (justify left) hide)
     )
-    (property "Footprint" "TestPoint:TestPoint_Pad_D1.0mm" (at 109.22 81.28 0)
-      (effects (font (size 1.27 1.27)) hide)
-    )
-    (property "Datasheet" "~" (at 109.22 81.28 0)
+    (property "Footprint" "TestPoint:TestPoint_Pad_D1.0mm" (at 109.22 91.44 0)
+      (effects (font (size 1.27 1.27)) hide)
+    )
+    (property "Datasheet" "~" (at 109.22 91.44 0)
       (effects (font (size 1.27 1.27)) hide)
     )
@@
     )
   )
-  (symbol (lib_id "Connector:TestPoint") (at 109.22 73.66 270) (unit 1)
+  (symbol (lib_id "Connector:TestPoint") (at 109.22 83.82 270) (unit 1)
     (in_bom yes) (on_board yes) (dnp no)
-    (property "Reference" "TP5" (at 114.3 73.025 90)
-      (effects (font (size 1.27 1.27)) (justify left))
-    )
-    (property "Value" "TestPoint" (at 118.11 73.66 90)
+    (property "Reference" "TP5" (at 114.3 83.185 90)
+      (effects (font (size 1.27 1.27)) (justify left))
+    )
+    (property "Value" "TestPoint" (at 118.11 83.82 90)
       (effects (font (size 1.27 1.27)) (justify left) hide)
     )
-    (property "Footprint" "TestPoint:TestPoint_Pad_D1.0mm" (at 109.22 78.74 0)
-      (effects (font (size 1.27 1.27)) hide)
-    )
-    (property "Datasheet" "~" (at 109.22 78.74 0)
-      (effects (font (size 1.27 1.27)) hide)
-    )
+    (property "Footprint" "TestPoint:TestPoint_Pad_D1.0mm" (at 109.22 88.9 0)
+      (effects (font (size 1.27 1.27)) hide)
+    )
+    (property "Datasheet" "~" (at 109.22 88.9 0)
+      (effects (font (size 1.27 1.27)) hide)
+    )
